File: tow_car.kicad_pcb (KiCad board)
At the start: 2 copper layers, 94 x 61.8 mm, 36 parts, among them J1 Conn_01x04_Male, J10 Conn_01x04_Male, J11 Conn_01x01_Male, J12 Conn_01x01, J13 Conn_01x02_Male, J14 Conn_01x01_Male, J15 Conn_01x03, J16 Conn_01x04_Male, J17 Conn_01x04_Male, J2 Conn_01x04_Male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

Commit message: Misc updates
Parts:
- added ?: , , F.Cu at (233.8, 115.6)
- added ?: , , F.Cu at (232.9, 115.4)
- added ?: , , F.Cu at (233.7, 115.6)
- added ?: , , F.Cu at (233.4, 115.6)
- moved C1 6.35 mm to (238.8, 97.2), turned to 90 degrees
- moved C5 4.01 mm to (240.4, 102.8), turned to 270 degrees
- moved R4 2.37 mm to (238.4, 91.7)
Connections:
- J17 pad 1: Net-(J13-Pad1) -> Net-(J17-Pad1)
- J17 pad 3: Net-(J17-Pad3) -> Net-(J13-Pad1)
- U2 pad : (no net) -> GND
- U2 pad 6: Net-(J17-Pad4) -> Net-(J17-Pad1)
- U2 pad 8: Net-(J17-Pad3) -> Net-(J17-Pad4)
Routing:
- net Net-(J17-Pad3): track 18.0 -> 0.00 mm
- net Net-(J17-Pad1): track 0.00 -> 17.2 mm
- net Net-(C1-Pad1): track 29.2 -> 34.8 mm
- net Net-(J13-Pad1): track 35.0 -> 30.3 mm
- net GND: track 70.2 -> 74.9 mm, vias 2 -> 7
- net Net-(U1-Pad10): track 43.0 -> 46.0 mm
- net Net-(U1-Pad9): track 47.9 -> 50.7 mm
- net +3V3: track 72.1 -> 72.9 mm
- net Net-(J17-Pad4): track 13.6 -> 13.8 mm, vias 1 -> 0
- net Net-(J16-Pad1): vias 5 -> 4
Other:
- board text added: "+"
- board text added: "1: OUT1 4: OUT2"
- board text added: "out1"
- board text added: "out2"
- board text removed: "-"

Commit message: Mupp
Connections:
- U2 pad : GND -> (no net)
Other:
- board text added: "+9V"
- board text removed: "+"

Commit message: Clean up
Parts:
- added J4: Conn_01x02_Male, Connector_PinHeader_2.54mm:PinHeader_2x01_P2.54mm_Vertical, F.Cu at (170.8, 88.3)
- C5: footprint Capacitor_SMD:CP_Elec_3x5.3 -> Capacitor_SMD:CP_Elec_6.3x3.9
- moved J12 4.28 mm to (232.6, 111.0)
- moved C5 3.93 mm to (236.5, 103.5), turned to 180 degrees
- moved J17 0.26 mm to (243.1, 113.2)
Connections:
- J2 pad 1: Net-(J2-Pad1) -> GND
- J2 pad 4: GND -> Net-(J2-Pad4)
- J5 pad 2: Net-(J2-Pad1) -> Net-(J2-Pad4)
- U2 pad : (no net) -> GND
Routing:
- net Net-(J2-Pad4): track 0.00 -> 46.0 mm
- net Net-(J2-Pad1): track 43.0 -> 0.00 mm
- net GND: track 74.9 -> 82.3 mm, vias 7 -> 5
- net Net-(C1-Pad1): track 34.8 -> 37.5 mm
- net Net-(U1-Pad10): track 46.0 -> 44.8 mm
- net Net-(J12-Pad1): track 15.9 -> 17.0 mm
- net Net-(J17-Pad4): track 13.8 -> 14.6 mm
- net Net-(U1-Pad9): track 50.7 -> 50.0 mm
- net Net-(J13-Pad1): track 30.3 -> 29.8 mm
